File: schematics/wall_terminal/wall_terminal.kicad_pcb (KiCad board)
At the start: 2 copper layers, 34.5 x 42.9 mm, 23 parts, among them J1 6P6C, J2 6P6C, J3 Conn_02x12_Odd_Even, Q1 2N7000, U1 ATtiny13A-P, U2 MAX487E

Commit message: !feat: first wall terminal PCB prototype.
Parts:
- removed the R10 at (149.8, 51.6)
- added J4: Reset, Connector_PinHeader_2.54mm:PinHeader_1x02_P2.54mm_Vertical, F.Cu at (171.7, 60.8)
- added REF**: SolderJumper-3_P1.3mm_Open_Pad1.0x1.5mm, Jumper:SolderJumper-3_P1.3mm_Open_Pad1.0x1.5mm, B.Cu at (176.5, 81.8)
- added REF**: SolderJumper-3_P1.3mm_Open_Pad1.0x1.5mm, Jumper:SolderJumper-3_P1.3mm_Open_Pad1.0x1.5mm, B.Cu at (176.5, 84.6)
- added REF**: SolderJumper-3_P1.3mm_Open_Pad1.0x1.5mm, Jumper:SolderJumper-3_P1.3mm_Open_Pad1.0x1.5mm, B.Cu at (147.5, 81.8)
- added REF**: SolderJumper-3_P1.3mm_Open_Pad1.0x1.5mm, Jumper:SolderJumper-3_P1.3mm_Open_Pad1.0x1.5mm, B.Cu at (147.5, 84.6)
- moved R10 4.75 mm to (149.6, 55.4)
- moved J3 4.04 mm to (149.4, 52.0)
- moved R3 3.84 mm to (171.1, 55.4)
- moved R2 3.84 mm to (174.2, 55.4)
- moved R1 3.84 mm to (177.3, 55.4)
- moved R9 3.81 mm to (152.7, 55.4)
- moved R8 3.81 mm to (155.8, 55.4)
- moved R7 3.81 mm to (158.8, 55.4)
- moved R6 3.81 mm to (161.9, 55.4)
- moved R5 3.81 mm to (165.0, 55.4)
- moved R4 3.81 mm to (168.1, 55.4)
- moved Q1 2.05 mm to (175.0, 62.8)
- moved C2 1.38 mm to (169.2, 68.9)
- moved C1 0.74 mm to (172.5, 67.8)
- renumbered R11 to R10, R12 to R11
Connections:
- R10 pad 1: /LED+ -> +5V
- R10 pad 2: +5V -> /LED+
- R11 pad 1: /RS485_A -> /RS485_B
- R11 pad 2: /RS485_B -> /RS485_A
- U1 pad 1: unconnected-(U1-~{RESET}/PB5-Pad1) -> Net-(J4-Pin_2)
Routing:
- net +5V: track 0.00 -> 77.4 mm
- net /LED-: track 0.00 -> 45.4 mm
- net /RS485_B: track 0.00 -> 38.4 mm
- net /RS485_A: track 0.00 -> 32.2 mm
- net /BUS_SHORT_6: track 0.00 -> 28.6 mm
- net Net-(JP1-C): track 0.00 -> 28.5 mm
- net Net-(JP2-C): track 0.00 -> 19.3 mm
- net /BUS_SHORT_1: track 0.00 -> 14.1 mm, vias 0 -> 1
- net /PB4: track 0.00 -> 12.1 mm
- net /PB3: track 0.00 -> 12.1 mm
- net /PB2: track 0.00 -> 9.73 mm, vias 0 -> 1
- net Net-(J4-Pin_2): track 0.00 -> 9.26 mm
- net /LED+: track 0.00 -> 9.13 mm
- net /PB0: track 0.00 -> 7.03 mm
- net /PB1: track 0.00 -> 5.75 mm
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- added copper zone on B.Cu, net GND
Other:
- board size 34.5 x 42.9 mm -> 34.5 x 39.4 mm
- board text added: "IN Analog OUT PWM"
- board text added: "IN Interrrupt OUT High/Low"
