File: hardware/schematics/control_unit/mcu.kicad_sch (KiCad schematic)
At the start: 2 parts

Commit message: fix
Connections:
- net OUT_4: now also U1.22 (G22); no longer U1.21 (G23)
- net OUT_5: now also U1.21 (G23); no longer U1.22 (G22)
