File: hardware/schematics/control_unit/mcu.kicad_sch (KiCad schematic)
At the start: 2 parts

Commit message: chore
Parts:
- renumbered C5 to C1, U1 to U12
Changed lines of the file:
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@@
 		(dnp no)
 		(fields_autoplaced yes)
-		(property "Reference" "U1"
+		(property "Reference" "U12"
 			(at 111.76 78.7714 0)
 			(effects
@@
 			(project "control_unit"
 				(path "/95f83be4-8e7e-4d00-b795-d60cd8e47b85/7664bf1e-4b5c-43ea-a123-dd981a1854d7"
-					(reference "U1")
+					(reference "U12")
 					(unit 1)
 				)
@@
 		(dnp no)
 		(fields_autoplaced yes)
-		(property "Reference" "C5"
+		(property "Reference" "C1"
 			(at 129.54 37.2109 0)
 			(effects
@@
 			(project "control_unit"
 				(path "/95f83be4-8e7e-4d00-b795-d60cd8e47b85/7664bf1e-4b5c-43ea-a123-dd981a1854d7"
-					(reference "C5")
+					(reference "C1")
 					(unit 1)
 				)

Commit message: !refactor
Connections:
- net OUT_1 renamed O1
- net OUT_10 renamed O10
- net OUT_2 renamed O2
- net OUT_3 renamed O3
- net OUT_4 renamed O4
- net OUT_5 renamed O5
- net OUT_6 renamed O6
- net OUT_7 renamed O7
- net OUT_8 renamed O8
- net OUT_9 renamed O9
- net RESET renamed ~{RST}
- net RTS renamed DE/~{RE}
- net RXD renamed RX
- net TXD renamed TX
Changed lines of the file:
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@@
 		)
 	)
-	(hierarchical_label "RXD"
+	(hierarchical_label "RX"
 		(shape input)
 		(at 137.16 77.47 0)
@@
 		)
 	)
-	(hierarchical_label "OUT_3"
+	(hierarchical_label "O3"
 		(shape input)
 		(at 137.16 87.63 0)
@@
 		)
 	)
-	(hierarchical_label "RESET"
+	(hierarchical_label "~{RST}"
 		(shape input)
 		(at 111.76 83.82 180)
@@
 		)
 	)
-	(hierarchical_label "OUT_6"
+	(hierarchical_label "O6"
 		(shape input)
 		(at 137.16 95.25 0)
@@
 		)
 	)
-	(hierarchical_label "TXD"
+	(hierarchical_label "TX"
 		(shape input)
 		(at 137.16 80.01 0)
@@
 		)
 	)
-	(hierarchical_label "OUT_9"
+	(hierarchical_label "O9"
 		(shape input)
 		(at 137.16 102.87 0)
@@
 		)
 	)
-	(hierarchical_label "OUT_8"
+	(hierarchical_label "O8"
 		(shape input)
 		(at 137.16 100.33 0)
@@
 		)
 	)
-	(hierarchical_label "RTS"
+	(hierarchical_label "DE{slash}~{RE}"
 		(shape input)
 		(at 137.16 69.85 0)
@@
 		)
 	)
-	(hierarchical_label "OUT_10"
+	(hierarchical_label "O10"
 		(shape input)
 		(at 137.16 105.41 0)
@@
 		)
 	)
-	(hierarchical_label "OUT_5"
+	(hierarchical_label "O5"
 		(shape input)
 		(at 137.16 92.71 0)
@@
 		)
 	)
-	(hierarchical_label "OUT_7"
+	(hierarchical_label "O7"
 		(shape input)
 		(at 137.16 97.79 0)
@@
 		)
 	)
-	(hierarchical_label "OUT_1"
+	(hierarchical_label "O1"
 		(shape input)
 		(at 137.16 82.55 0)
@@
 		)
 	)
-	(hierarchical_label "OUT_4"
+	(hierarchical_label "O4"
 		(shape input)
 		(at 137.16 90.17 0)
@@
 		)
 	)
-	(hierarchical_label "OUT_2"
+	(hierarchical_label "O2"
 		(shape input)
 		(at 137.16 85.09 0)

Commit message: feat
Parts:
- renumbered U12 to U14
Connections:
- net DE/~{RE}: now also U14.7 (G12); no longer U14.5 (G13)
- net O1: now also U14.32 (G4); no longer U14.28 (G18)
- net O10: now also U14.11 (G25); no longer U14.12 (G33)
- net O2: now also U14.5 (G13); no longer U14.27 (G19)
- net O3: now also U14.31 (G16); no longer U14.25 (G21)
- net O4: now also U14.30 (G17); no longer U14.22 (G22)
- net O5: now also U14.28 (G18); no longer U14.21 (G23)
- net O6: now also U14.27 (G19); no longer U14.11 (G25)
- net O7: now also U14.25 (G21); no longer U14.10 (G26)
- net O8: now also U14.22 (G22); no longer U14.9 (G27)
- net O9: now also U14.21 (G23); no longer U14.13 (G32)
- net RX: now also U14.15 (G34); no longer U14.31 (G16)
- net TX: now also U14.29 (G5); no longer U14.30 (G17)
- net O18: now reaches U14.33 (G0)
- net O17: now reaches U14.34 (G2)
- net O16: now reaches U14.35 (G15)
- net O15: now reaches U14.8 (G14)
- net ~{RST}: no longer names the net of U14.18 (EN/~{RESET})
- new net O11: U14.10 (G26)
- new net O12: U14.9 (G27)
- new net O13: U14.13 (G32)
- new net O14: U14.12 (G33)
- no-connect marks 13 -> 6
Changed lines of the file:
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@@
-	)
-	(no_connect
-		(at 137.16 107.95)
 	)
 	(no_connect
@@
 	)
 	(no_connect
-		(at 137.16 74.93)
-	)
-	(no_connect
 		(at 137.16 59.69)
 	)
@@
 	)
 	(no_connect
-		(at 137.16 57.15)
-	)
-	(no_connect
-		(at 137.16 64.77)
-	)
-	(no_connect
-		(at 137.16 52.07)
-	)
-	(no_connect
-		(at 137.16 67.31)
+		(at 111.76 83.82)
 	)
 	(no_connect
 		(at 137.16 110.49)
-	)
-	(no_connect
-		(at 137.16 62.23)
-	)
-	(no_connect
-		(at 137.16 72.39)
 	)
 	(no_connect
@@
 	(hierarchical_label "RX"
 		(shape input)
+		(at 137.16 107.95 0)
+		(fields_autoplaced yes)
+		(effects
+			(font
+				(size 1.27 1.27)
+			)
+			(justify left)
+		)
+	)
+	(hierarchical_label "O3"
+		(shape input)
 		(at 137.16 77.47 0)
 		(fields_autoplaced yes)
@@
 		)
 	)
-	(hierarchical_label "O3"
+	(hierarchical_label "O6"
+		(shape input)
+		(at 137.16 85.09 0)
+		(fields_autoplaced yes)
+		(effects
+			(font
+				(size 1.27 1.27)
+			)
+			(justify left)
+		)
+	)
+	(hierarchical_label "O12"
+		(shape input)
+		(at 137.16 100.33 0)
+		(fields_autoplaced yes)
+		(effects
+			(font
+				(size 1.27 1.27)
+			)
+			(justify left)
+		)
+	)
+	(hierarchical_label "O18"
+		(shape input)
+		(at 137.16 52.07 0)
+		(fields_autoplaced yes)
+		(effects
+			(font
+				(size 1.27 1.27)
+			)
+			(justify left)
+		)
+	)
+	(hierarchical_label "O16"
+		(shape input)
+		(at 137.16 74.93 0)
+		(fields_autoplaced yes)
+		(effects
+			(font
+				(size 1.27 1.27)
+			)
+			(justify left)
+		)
+	)
+	(hierarchical_label "TX"
+		(shape input)
+		(at 137.16 64.77 0)
+		(fields_autoplaced yes)
+		(effects
+			(font
+				(size 1.27 1.27)
+			)
+			(justify left)
+		)
+	)
+	(hierarchical_label "O9"
+		(shape input)
+		(at 137.16 92.71 0)
+		(fields_autoplaced yes)
+		(effects
+			(font
+				(size 1.27 1.27)
+			)
+			(justify left)
+		)
+	)
+	(hierarchical_label "O13"
+		(shape input)
+		(at 137.16 102.87 0)
+		(fields_autoplaced yes)
+		(effects
+			(font
+				(size 1.27 1.27)
+			)
+			(justify left)
+		)
+	)
+	(hierarchical_label "O11"
+		(shape input)
+		(at 137.16 97.79 0)
+		(fields_autoplaced yes)
+		(effects
+			(font
+				(size 1.27 1.27)
+			)
+			(justify left)
+		)
+	)
+	(hierarchical_label "O8"
+		(shape input)
+		(at 137.16 90.17 0)
+		(fields_autoplaced yes)
+		(effects
+			(font
+				(size 1.27 1.27)
+			)
+			(justify left)
+		)
+	)
+	(hierarchical_label "DE{slash}~{RE}"
+		(shape input)
+		(at 137.16 67.31 0)
+		(fields_autoplaced yes)
+		(effects
+			(font
+				(size 1.27 1.27)
+			)
+			(justify left)
+		)
+	)
+	(hierarchical_label "O10"
+		(shape input)
+		(at 137.16 95.25 0)
+		(fields_autoplaced yes)
+		(effects
+			(font
+				(size 1.27 1.27)
+			)
+			(justify left)
+		)
+	)
+	(hierarchical_label "O5"
+		(shape input)
+		(at 137.16 82.55 0)
+		(fields_autoplaced yes)
+		(effects
+			(font
+				(size 1.27 1.27)
+			)
+			(justify left)
+		)
+	)
+	(hierarchical_label "O17"
+		(shape input)
+		(at 137.16 57.15 0)
+		(fields_autoplaced yes)
+		(effects
+			(font
+				(size 1.27 1.27)
+			)
+			(justify left)
+		)
+	)
+	(hierarchical_label "O7"
 		(shape input)
 		(at 137.16 87.63 0)
@@
 		)
 	)
-	(hierarchical_label "~{RST}"
-		(shape input)
-		(at 111.76 83.82 180)
+	(hierarchical_label "O1"
+		(shape input)
+		(at 137.16 62.23 0)
+		(fields_autoplaced yes)
+		(effects
+			(font
+				(size 1.27 1.27)
+			)
+			(justify left)
+		)
+	)
+	(hierarchical_label "GND"
+		(shape input)
+		(at 125.73 43.18 270)
 		(fields_autoplaced yes)
 		(effects
@@
 		)
 	)
-	(hierarchical_label "O6"
-		(shape input)
-		(at 137.16 95.25 0)
-		(fields_autoplaced yes)
-		(effects
-			(font
-				(size 1.27 1.27)
-			)
-			(justify left)
-		)
-	)
-	(hierarchical_label "TX"
+	(hierarchical_label "O4"
 		(shape input)
 		(at 137.16 80.01 0)
@@
 		)
 	)
-	(hierarchical_label "O9"
-		(shape input)
-		(at 137.16 102.87 0)
-		(fields_autoplaced yes)
-		(effects
-			(font
-				(size 1.27 1.27)
-			)
-			(justify left)
-		)
-	)
-	(hierarchical_label "O8"
-		(shape input)
-		(at 137.16 100.33 0)
-		(fields_autoplaced yes)
-		(effects
-			(font
-				(size 1.27 1.27)
-			)
-			(justify left)
-		)
-	)
-	(hierarchical_label "DE{slash}~{RE}"
+	(hierarchical_label "O14"
+		(shape input)
+		(at 137.16 105.41 0)
+		(fields_autoplaced yes)
+		(effects
+			(font
+				(size 1.27 1.27)
+			)
+			(justify left)
+		)
+	)
+	(hierarchical_label "O2"
 		(shape input)
 		(at 137.16 69.85 0)
@@
 		)
 	)
-	(hierarchical_label "O10"
-		(shape input)
-		(at 137.16 105.41 0)
-		(fields_autoplaced yes)
-		(effects
-			(font
-				(size 1.27 1.27)
-			)
-			(justify left)
-		)
-	)
-	(hierarchical_label "O5"
-		(shape input)
-		(at 137.16 92.71 0)
-		(fields_autoplaced yes)
-		(effects
-			(font
-				(size 1.27 1.27)
-			)
-			(justify left)
-		)
-	)
-	(hierarchical_label "O7"
-		(shape input)
-		(at 137.16 97.79 0)
-		(fields_autoplaced yes)
-		(effects
-			(font
-				(size 1.27 1.27)
-			)
-			(justify left)
-		)
-	)
-	(hierarchical_label "O1"
-		(shape input)
-		(at 137.16 82.55 0)
-		(fields_autoplaced yes)
-		(effects
-			(font
-				(size 1.27 1.27)
-			)
-			(justify left)
-		)
-	)
 	(hierarchical_label "GND"
 		(shape input)
-		(at 125.73 43.18 270)
+		(at 124.46 120.65 270)
 		(fields_autoplaced yes)
 		(effects
@@
 		)
 	)
-	(hierarchical_label "O4"
-		(shape input)
-		(at 137.16 90.17 0)
-		(fields_autoplaced yes)
-		(effects
-			(font
-				(size 1.27 1.27)
-			)
-			(justify left)
-		)
-	)
-	(hierarchical_label "O2"
-		(shape input)
-		(at 137.16 85.09 0)
-		(fields_autoplaced yes)
-		(effects
-			(font
-				(size 1.27 1.27)
-			)
-			(justify left)
-		)
-	)
-	(hierarchical_label "GND"
-		(shape input)
-		(at 124.46 120.65 270)
-		(fields_autoplaced yes)
-		(effects
-			(font
-				(size 1.27 1.27)
-			)
-			(justify right)
+	(hierarchical_label "O15"
+		(shape input)
+		(at 137.16 72.39 0)
+		(fields_autoplaced yes)
+		(effects
+			(font
+				(size 1.27 1.27)
+			)
+			(justify left)
 		)
 	)
@@
 		(dnp no)
 		(fields_autoplaced yes)
-		(property "Reference" "U12"
+		(property "Reference" "U14"
 			(at 111.76 78.7714 0)
 			(effects
@@
 			(project "control_unit"
 				(path "/95f83be4-8e7e-4d00-b795-d60cd8e47b85/7664bf1e-4b5c-43ea-a123-dd981a1854d7"
-					(reference "U12")
+					(reference "U14")
 					(unit 1)
 				)

Commit message: !feat
Connections:
- net O18 is gone; now on net DE/~{RE}: U14.33 (G0)
- net DE/~{RE}: no longer U14.7 (G12)
- net O11: now also U14.35 (G15); no longer U14.10 (G26)
- net O12: now also U14.29 (G5); no longer U14.9 (G27)
- net O13: now also U14.10 (G26); no longer U14.13 (G32)
- net O14: now also U14.9 (G27); no longer U14.12 (G33)
- net O15: now also U14.13 (G32); no longer U14.8 (G14)
- net O16: now also U14.7 (G12); no longer U14.35 (G15)
- net O17: now also U14.8 (G14); no longer U14.34 (G2)
- net TX: now also U14.34 (G2); no longer U14.29 (G5)
- net TEMP: now reaches U14.14 (G35)
- net AC_I: now reaches U14.16 (SN/G39)
- net AC_V: now reaches U14.17 (SP/G36)
- net 3.3V: now reaches C1.1, U14.19 (3V3)
- new net FAN: U14.12 (G33)
- no-connect marks 6 -> 3

Commit message: feat
Parts:
- removed U14: ~, MCU_Espressif_ESP32_38PIN:ESP32_38PIN, symbol MCU_Espressif_ESP32_38PIN:ESP32_38PIN_Ideal
- added U15: ESP-WROOM-32, MCU_Espressif_ESP32_38PIN:ESP32_38PIN, symbol MCU_Espressif_ESP32_38PIN:ESP32_38PIN_Ideal
- C1: footprint (none) -> Capacitor_THT:CP_Radial_D6.3mm_P2.50mm
Connections:
- net 3.3V: now also U15.19 (3V3)
- net 5V: now also U15.1 (V5/Vin)
- net AC_I: now also U15.16 (SN/G39)
- net AC_V: now also U15.17 (SP/G36)
- net DE/~{RE}: now also U15.33 (G0)
- net FAN: now also U15.12 (G33)
- net GND: now also U15.20 (GND), U15.26 (GND), U15.6 (GND)
- net O1: now also U15.32 (G4)
- net O10: now also U15.11 (G25)
- net O11: now also U15.35 (G15)
- net O12: now also U15.29 (G5)
- net O13: now also U15.10 (G26)
- net O14: now also U15.9 (G27)
- net O15: now also U15.13 (G32)
- net O16: now also U15.7 (G12)
- net O2: now also U15.5 (G13)
- net O3: now also U15.31 (G16)
- net O4: now also U15.30 (G17)
- net O5: now also U15.28 (G18)
- net O6: now also U15.27 (G19)
- net O7: now also U15.25 (G21)
- net O8: now also U15.22 (G22)
- net O9: now also U15.21 (G23)
- net RX: now also U15.15 (G34)
- net TEMP: now also U15.14 (G35)
- net TX: now also U15.34 (G2)
- new net ALARM: U15.8 (G14)
Changed lines of the file:
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@@
 		)
 	)
-	(hierarchical_label "O17"
+	(hierarchical_label "ALARM"
 		(shape input)
 		(at 137.16 72.39 0)
@@
 			)
 			(justify left)
-		)
-	)
-	(hierarchical_label "3.3V"
-		(shape input)
-		(at 74.93 50.8 180)
-		(fields_autoplaced yes)
-		(effects
-			(font
-				(size 1.27 1.27)
-			)
-			(justify right)
 		)
 	)
@@
 		(dnp no)
 		(fields_autoplaced yes)
-		(property "Reference" "U14"
-			(at 111.76 78.7714 0)
-			(effects
-				(font
-					(size 1.27 1.27)
-				)
-			)
-		)
-		(property "Value" "~"
-			(at 111.76 80.6765 0)
+		(property "Reference" "U15"
+			(at 105.41 77.5014 0)
+			(effects
+				(font
+					(size 1.27 1.27)
+				)
+			)
+		)
+		(property "Value" "ESP-WROOM-32"
+			(at 105.41 80.0414 0)
 			(effects
 				(font
@@
 			)
 		)
+		(pin "16"
+		)
+		(pin "10"
+		)
+		(pin "12"
+		)
+		(pin "32"
+		)
+		(pin "35"
+		)
+		(pin "24"
+		)
+		(pin "18"
+		)
+		(pin "3"
+		)
+		(pin "19"
+		)
+		(pin "26"
+		)
+		(pin "22"
+		)
+		(pin "31"
+		)
+		(pin "37"
+		)
+		(pin "9"
+		)
+		(pin "5"
+		)
+		(pin "1"
+		)
+		(pin "11"
+		)
+		(pin "14"
+		)
+		(pin "2"
+		)
+		(pin "27"
+		)
+		(pin "17"
+		)
+		(pin "36"
+		)
+		(pin "38"
+		)
+		(pin "28"
+		)
 		(pin "13"
 		)
+		(pin "33"
+		)
+		(pin "7"
+		)
+		(pin "23"
+		)
+		(pin "25"
+		)
+		(pin "29"
+		)
+		(pin "21"
+		)
 		(pin "20"
 		)
-		(pin "27"
-		)
-		(pin "36"
-		)
-		(pin "29"
-		)
-		(pin "9"
-		)
-		(pin "37"
-		)
-		(pin "18"
-		)
-		(pin "26"
-		)
-		(pin "17"
-		)
-		(pin "28"
-		)
-		(pin "31"
-		)
-		(pin "35"
+		(pin "34"
+		)
+		(pin "4"
+		)
+		(pin "30"
+		)
+		(pin "6"
 		)
 		(pin "15"
 		)
-		(pin "2"
-		)
-		(pin "11"
-		)
-		(pin "33"
-		)
-		(pin "22"
-		)
-		(pin "30"
-		)
-		(pin "10"
-		)
-		(pin "7"
-		)
-		(pin "5"
-		)
-		(pin "6"
-		)
-		(pin "1"
-		)
-		(pin "34"
-		)
-		(pin "14"
-		)
-		(pin "3"
-		)
 		(pin "8"
-		)
-		(pin "32"
-		)
-		(pin "25"
-		)
-		(pin "16"
-		)
-		(pin "4"
-		)
-		(pin "12"
-		)
-		(pin "19"
-		)
-		(pin "23"
-		)
-		(pin "21"
-		)
-		(pin "24"
-		)
-		(pin "38"
-		)
-		(instances
-			(project "control_unit"
-				(path "/95f83be4-8e7e-4d00-b795-d60cd8e47b85/7664bf1e-4b5c-43ea-a123-dd981a1854d7"
-					(reference "U14")
-					(unit 1)
-				)
-			)
-		)
-	)
-	(symbol
-		(lib_id "power:PWR_FLAG")
-		(at 74.93 50.8 270)
-		(unit 1)
-		(exclude_from_sim no)
-		(in_bom yes)
-		(on_board yes)
-		(dnp no)
-		(fields_autoplaced yes)
-		(property "Reference" "#FLG04"
-			(at 76.835 50.8 0)
-			(effects
-				(font
-					(size 1.27 1.27)
-				)
-				(hide yes)
-			)
-		)
-		(property "Value" "PWR_FLAG"
-			(at 78.74 50.8001 90)
-			(effects
-				(font
-					(size 1.27 1.27)
-				)
-				(justify left)
-			)
-		)
-		(property "Footprint" ""
-			(at 74.93 50.8 0)
-			(effects
-				(font
-					(size 1.27 1.27)
-				)
-				(hide yes)
-			)
-		)
-		(property "Datasheet" "~"
-			(at 74.93 50.8 0)
-			(effects
-				(font
-					(size 1.27 1.27)
-				)
-				(hide yes)
-			)
-		)
-		(property "Description" "Special symbol for telling ERC where power comes from"
-			(at 74.93 50.8 0)
-			(effects
-				(font
-					(size 1.27 1.27)
-				)
-				(hide yes)
-			)
-		)
-		(pin "1"
 		)
 		(instances
 			(project ""
 				(path "/95f83be4-8e7e-4d00-b795-d60cd8e47b85/7664bf1e-4b5c-43ea-a123-dd981a1854d7"
-					(reference "#FLG04")
+					(reference "U15")
 					(unit 1)
 				)
@@
 			)
 		)
-		(property "Footprint" ""
+		(property "Footprint" "Capacitor_THT:CP_Radial_D6.3mm_P2.50mm"
 			(at 100.0252 54.61 0)
 			(effects

Commit message: !feat
Connections:
- net ~{RESET}: now reaches U15.18 (EN/~{RESET})
- no-connect marks 3 -> 2
Changed lines of the file:
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@@
 		(at 137.16 59.69)
-	)
-	(no_connect
-		(at 111.76 83.82)
 	)
 	(hierarchical_label "5V"
@@
 		)
 	)
+	(hierarchical_label "~{RESET}"
+		(shape input)
+		(at 111.76 83.82 180)
+		(fields_autoplaced yes)
+		(effects
+			(font
+				(size 1.27 1.27)
+			)
+			(justify right)
+		)
+	)
