File: hardware/schematics/control_unit/control_unit.kicad_sch (KiCad schematic)
At the start: 2 parts, among them J1 6P6C

Commit message: chore
Other:
- note added: "NOTE: Chiedere se predisporre anche uscite per relay Predisporre gruppo di continuita'"
- note removed: "NOTE: Chiedere se predisporre anche uscite per relay"
Changed lines of the file:
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@@
 		)
 	)
-	(text "NOTE:\nChiedere se predisporre anche uscite per relay"
+	(text "NOTE:\nChiedere se predisporre anche uscite per relay\nPredisporre gruppo di continuita'"
 		(exclude_from_sim no)
 		(at 146.558 29.718 0)

Commit message: chore
Other:
- note added: "NOTE: Chiedere se predisporre anche uscite per relay"
- note removed: "NOTE: Chiedere se predisporre anche uscite per relay Predisporre gruppo di continuita'"
Changed lines of the file:
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@@
 		)
 	)
-	(text "NOTE:\nChiedere se predisporre anche uscite per relay\nPredisporre gruppo di continuita'"
+	(text "NOTE:\nChiedere se predisporre anche uscite per relay"
 		(exclude_from_sim no)
 		(at 146.558 29.718 0)
@@
 		(dnp no)
 		(fields_autoplaced yes)
-		(property "Reference" "#PWR010"
+		(property "Reference" "#PWR011"
 			(at 121.92 29.21 0)
 			(effects
@@
 			(project "control_unit"
 				(path "/95f83be4-8e7e-4d00-b795-d60cd8e47b85"
-					(reference "#PWR010")
+					(reference "#PWR011")
 					(unit 1)
 				)
@@
 		(dnp no)
 		(fields_autoplaced yes)
-		(property "Reference" "#PWR011"
+		(property "Reference" "#PWR010"
 			(at 115.57 67.31 0)
 			(effects
@@
 			(project "control_unit"
 				(path "/95f83be4-8e7e-4d00-b795-d60cd8e47b85"
-					(reference "#PWR011")
+					(reference "#PWR010")
 					(unit 1)
 				)
@@
 		(dnp no)
 		(fields_autoplaced yes)
-		(property "Reference" "#PWR08"
+		(property "Reference" "#PWR07"
 			(at 92.71 58.42 0)
 			(effects
@@
 			(project "control_unit"
 				(path "/95f83be4-8e7e-4d00-b795-d60cd8e47b85"
-					(reference "#PWR08")
+					(reference "#PWR07")
 					(unit 1)
 				)
@@
 		(dnp no)
 		(fields_autoplaced yes)
-		(property "Reference" "#PWR012"
+		(property "Reference" "#PWR09"
 			(at 109.22 77.47 0)
 			(effects
@@
 			(project "control_unit"
 				(path "/95f83be4-8e7e-4d00-b795-d60cd8e47b85"
-					(reference "#PWR012")
+					(reference "#PWR09")
 					(unit 1)
 				)
@@
 		(dnp no)
 		(fields_autoplaced yes)
-		(property "Reference" "#PWR07"
+		(property "Reference" "#PWR06"
 			(at 82.55 86.36 0)
 			(effects
@@
 			(project "control_unit"
 				(path "/95f83be4-8e7e-4d00-b795-d60cd8e47b85"
-					(reference "#PWR07")
+					(reference "#PWR06")
 					(unit 1)
 				)
@@
 		(dnp no)
 		(fields_autoplaced yes)
-		(property "Reference" "#PWR06"
+		(property "Reference" "#PWR08"
 			(at 99.06 81.28 0)
 			(effects
@@
 			(project "control_unit"
 				(path "/95f83be4-8e7e-4d00-b795-d60cd8e47b85"
-					(reference "#PWR06")
+					(reference "#PWR08")
 					(unit 1)
 				)
@@
 		(dnp no)
 		(fields_autoplaced yes)
-		(property "Reference" "#PWR01"
+		(property "Reference" "#PWR02"
 			(at 31.75 40.64 0)
 			(effects
@@
 			(project "control_unit"
 				(path "/95f83be4-8e7e-4d00-b795-d60cd8e47b85"
-					(reference "#PWR01")
+					(reference "#PWR02")
 					(unit 1)
 				)
@@
 		(dnp no)
 		(fields_autoplaced yes)
-		(property "Reference" "#PWR09"
+		(property "Reference" "#PWR012"
 			(at 121.92 57.15 0)
 			(effects
@@
 			(project "control_unit"
 				(path "/95f83be4-8e7e-4d00-b795-d60cd8e47b85"
-					(reference "#PWR09")
+					(reference "#PWR012")
 					(unit 1)
 				)
@@
 		(dnp no)
 		(fields_autoplaced yes)
-		(property "Reference" "#PWR02"
+		(property "Reference" "#PWR01"
 			(at 29.21 26.67 0)
 			(effects
@@
 			(project "control_unit"
 				(path "/95f83be4-8e7e-4d00-b795-d60cd8e47b85"
-					(reference "#PWR02")
-					(unit 1)
-				)
+					(reference "#PWR01")
+					(unit 1)
+				)

Commit message: chore
Other:
- sheet PSU ports: added 24V, B+, B-; removed Vin
- note added: "NOTE: Chiedere se predisporre anche uscite per relay Predisporre ventola di raffreddamento e termocoppie Mettere fusibili Aggiungere altre zone con MOSFET (minimo 12)"
- note removed: "NOTE: Chiedere se predisporre anche uscite per relay"
Changed lines of the file:
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@@
 		)
 	)
-	(text "NOTE:\nChiedere se predisporre anche uscite per relay"
+	(text "NOTE:\nChiedere se predisporre anche uscite per relay\nPredisporre ventola di raffreddamento e termocoppie\nMettere fusibili\nAggiungere altre zone con MOSFET (minimo 12)"
 		(exclude_from_sim no)
 		(at 146.558 29.718 0)
@@
 	(symbol
 		(lib_id "power:GND")
-		(at 31.75 34.29 0)
+		(at 35.56 34.29 0)
 		(unit 1)
 		(exclude_from_sim no)
@@
 		(fields_autoplaced yes)
 		(property "Reference" "#PWR02"
-			(at 31.75 40.64 0)
+			(at 35.56 40.64 0)
 			(effects
 				(font
@@
 		)
 		(property "Value" "GND"
-			(at 31.75 39.37 0)
+			(at 35.56 39.37 0)
 			(effects
 				(font
@@
 		)
 		(property "Footprint" ""
-			(at 31.75 34.29 0)
+			(at 35.56 34.29 0)
 			(effects
 				(font
@@
 		)
 		(property "Datasheet" ""
-			(at 31.75 34.29 0)
+			(at 35.56 34.29 0)
 			(effects
 				(font
@@
 		)
 		(property "Description" "Power symbol creates a global label with name \"GND\" , ground"
-			(at 31.75 34.29 0)
+			(at 35.56 34.29 0)
 			(effects
 				(font
@@
 		)
 		(pin "GND" input
-			(at 31.75 34.29 270)
+			(at 35.56 34.29 270)
 			(effects
 				(font
@@
 			)
 		)
-		(pin "Vin" input
+		(pin "24V" input
 			(at 25.4 26.67 180)
 			(effects
 				(font
+					(size 1.27 1.27)
+				)
+				(justify left)
+			)
+		)
+		(pin "B-" input
+			(at 31.75 34.29 270)
+			(effects
+				(font
+					(size 1.27 1.27)
+				)
+				(justify left)
+			)
+		)
+		(pin "B+" input
+			(at 27.94 34.29 270)
+			(effects
+				(font

Commit message: !refactor
Connections:
- net PERIPHERALS/TX_EN renamed MCU/DE/~{RE}
- net PERIPHERALS/~{RX_EN} renamed PERIPHERALS/~{RE}
Other:
- sheet IN renamed PERIPHERALS
- sheet MCU ports: added DE/~{RE}, O1, O10, O2, O3, O4, O5, O6, O7, O8, O9, RX, TX, ~{RST}; removed OUT_1, OUT_10, OUT_2, OUT_3, OUT_4, OUT_5, OUT_6, OUT_7, OUT_8, OUT_9, RESET, RTS, RXD, TXD
- sheet OUT ports: added L1, L10, L2, L3, L4, L5, L6, L7, L8, L9, O1, O10, O2, O3, O4, O5, O6, O7, O8, O9; removed LED_1, LED_10, LED_2, LED_3, LED_4, LED_5, LED_6, LED_7, LED_8, LED_9, OUT_1, OUT_10, OUT_2, OUT_3, OUT_4, OUT_5, OUT_6, OUT_7, OUT_8, OUT_9
- sheet PERIPHERALS: file in.kicad_sch -> peripherals.kicad_sch
- sheet PERIPHERALS ports: added DE, RX, TX, ~{RE}; removed RXD, TXD, TX_EN, ~{RX_EN}
- sheet PSU ports: added none; removed B+, B-
Changed lines of the file:
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@@
 	(symbol
 		(lib_id "power:GND")
-		(at 67.31 71.12 0)
+		(at 66.04 71.12 0)
 		(unit 1)
 		(exclude_from_sim no)
@@
 		(fields_autoplaced yes)
 		(property "Reference" "#PWR05"
-			(at 67.31 77.47 0)
+			(at 66.04 77.47 0)
 			(effects
 				(font
@@
 		)
 		(property "Value" "GND"
-			(at 67.31 76.2 0)
+			(at 66.04 76.2 0)
 			(effects
 				(font
@@
 		)
 		(property "Footprint" ""
-			(at 67.31 71.12 0)
+			(at 66.04 71.12 0)
 			(effects
 				(font
@@
 		)
 		(property "Datasheet" ""
-			(at 67.31 71.12 0)
+			(at 66.04 71.12 0)
 			(effects
 				(font
@@
 		)
 		(property "Description" "Power symbol creates a global label with name \"GND\" , ground"
-			(at 67.31 71.12 0)
+			(at 66.04 71.12 0)
 			(effects
 				(font
@@
 	(symbol
 		(lib_id "power:GND")
-		(at 99.06 74.93 0)
+		(at 95.25 74.93 0)
 		(unit 1)
 		(exclude_from_sim no)
@@
 		(fields_autoplaced yes)
 		(property "Reference" "#PWR08"
-			(at 99.06 81.28 0)
+			(at 95.25 81.28 0)
 			(effects
 				(font
@@
 		)
 		(property "Value" "GND"
-			(at 99.06 80.01 0)
+			(at 95.25 80.01 0)
 			(effects
 				(font
@@
 		)
 		(property "Footprint" ""
-			(at 99.06 74.93 0)
+			(at 95.25 74.93 0)
 			(effects
 				(font
@@
 		)
 		(property "Datasheet" ""
-			(at 99.06 74.93 0)
+			(at 95.25 74.93 0)
 			(effects
 				(font
@@
 		)
 		(property "Description" "Power symbol creates a global label with name \"GND\" , ground"
-			(at 99.06 74.93 0)
+			(at 95.25 74.93 0)
 			(effects
 				(font
@@
 	(symbol
 		(lib_id "power:GND")
-		(at 35.56 34.29 0)
+		(at 31.75 34.29 0)
 		(unit 1)
 		(exclude_from_sim no)
@@
 		(fields_autoplaced yes)
 		(property "Reference" "#PWR02"
-			(at 35.56 40.64 0)
+			(at 31.75 40.64 0)
 			(effects
 				(font
@@
 		)
 		(property "Value" "GND"
-			(at 35.56 39.37 0)
+			(at 31.75 39.37 0)
 			(effects
 				(font
@@
 		)
 		(property "Footprint" ""
-			(at 35.56 34.29 0)
+			(at 31.75 34.29 0)
 			(effects
 				(font
@@
 		)
 		(property "Datasheet" ""
-			(at 35.56 34.29 0)
+			(at 31.75 34.29 0)
 			(effects
 				(font
@@
 		)
 		(property "Description" "Power symbol creates a global label with name \"GND\" , ground"
-			(at 35.56 34.29 0)
+			(at 31.75 34.29 0)
 			(effects
 				(font
@@
 			)
 		)
-		(pin "LED_10" input
+		(pin "L10" input
 			(at 132.08 49.53 0)
 			(effects
@@
 			)
 		)
-		(pin "OUT_10" input
+		(pin "O10" input
 			(at 111.76 49.53 180)
 			(effects
@@
 			)
 		)
-		(pin "OUT_9" input
+		(pin "O9" input
 			(at 111.76 46.99 180)
 			(effects
@@
 			)
 		)
-		(pin "LED_9" input
+		(pin "L9" input
 			(at 132.08 46.99 0)
 			(effects
@@
 			)
 		)
-		(pin "OUT_6" input
+		(pin "O6" input
 			(at 111.76 39.37 180)
 			(effects
@@
 			)
 		)
-		(pin "LED_4" input
+		(pin "L4" input
 			(at 132.08 34.29 0)
 			(effects
@@
 			)
 		)
-		(pin "LED_5" input
+		(pin "L5" input
 			(at 132.08 36.83 0)
 			(effects
@@
 			)
 		)
-		(pin "OUT_4" input
+		(pin "O4" input
 			(at 111.76 34.29 180)
 			(effects
@@
 			)
 		)
-		(pin "OUT_5" input
+		(pin "O5" input
 			(at 111.76 36.83 180)
 			(effects
@@
 			)
 		)
-		(pin "LED_2" input
+		(pin "L2" input
 			(at 132.08 29.21 0)
 			(effects
@@
 			)
 		)
-		(pin "LED_1" input
+		(pin "L1" input
 			(at 132.08 26.67 0)
 			(effects
@@
 			)
 		)
-		(pin "OUT_1" input
+		(pin "O1" input
 			(at 111.76 26.67 180)
 			(effects
@@
 			)
 		)
-		(pin "OUT_2" input
+		(pin "O2" input
 			(at 111.76 29.21 180)
 			(effects
@@
 			)
 		)
-		(pin "LED_3" input
+		(pin "L3" input
 			(at 132.08 31.75 0)
 			(effects
@@
 			)
 		)
-		(pin "LED_6" input
+		(pin "L6" input
 			(at 132.08 39.37 0)
 			(effects
@@
 			)
 		)
-		(pin "OUT_3" input
+		(pin "O3" input
 			(at 111.76 31.75 180)
 			(effects
@@
 			)
 		)
-		(pin "OUT_7" input
+		(pin "O7" input
 			(at 111.76 41.91 180)
 			(effects
@@
 			)
 		)
-		(pin "LED_7" input
+		(pin "L7" input
 			(at 132.08 41.91 0)
 			(effects
@@
 			)
 		)
-		(pin "OUT_8" input
+		(pin "O8" input
 			(at 111.76 44.45 180)
 			(effects
@@
 			)
 		)
-		(pin "LED_8" input
+		(pin "L8" input
 			(at 132.08 44.45 0)
 			(effects
@@
 		)
 		(pin "GND" input
-			(at 35.56 34.29 270)
+			(at 31.75 34.29 270)
 			(effects
 				(font
@@
 		(pin "24V" input
 			(at 25.4 26.67 180)
-			(effects
-				(font
-					(size 1.27 1.27)
-				)
-				(justify left)
-			)
-		)
-		(pin "B-" input
-			(at 31.75 34.29 270)
-			(effects
-				(font
-					(size 1.27 1.27)
-				)
-				(justify left)
-			)
-		)
-		(pin "B+" input
-			(at 27.94 34.29 270)
 			(effects
 				(font
@@
 			)
 		)
-		(pin "OUT_1" input
+		(pin "O1" input
 			(at 76.2 26.67 0)
 			(effects
@@
 			)
 		)
-		(pin "OUT_2" input
+		(pin "O2" input
 			(at 76.2 29.21 0)
 			(effects
@@
 			)
 		)
-		(pin "OUT_7" input
+		(pin "O7" input
 			(at 76.2 41.91 0)
 			(effects
@@
 			)
 		)
-		(pin "RXD" input
+		(pin "RX" input
 			(at 76.2 64.77 0)
 			(effects
@@
 			)
 		)
-		(pin "TXD" input
+		(pin "TX" input
 			(at 76.2 67.31 0)
 			(effects
@@
 			)
 		)
-		(pin "OUT_4" input
+		(pin "O4" input
 			(at 76.2 34.29 0)
 			(effects
@@
 			)
 		)
-		(pin "OUT_5" input
+		(pin "O5" input
 			(at 76.2 36.83 0)
 			(effects
@@
 			)
 		)
-		(pin "OUT_3" input
+		(pin "O3" input
 			(at 76.2 31.75 0)
 			(effects
@@
 			)
 		)
-		(pin "OUT_6" input
+		(pin "O6" input
 			(at 76.2 39.37 0)
 			(effects
@@
 		)
 		(pin "GND" input
-			(at 67.31 71.12 270)
-			(effects
-				(font
-					(size 1.27 1.27)
-				)
-				(justify left)
-			)
-		)
-		(pin "OUT_9" input
+			(at 66.04 71.12 270)
+			(effects
+				(font
+					(size 1.27 1.27)
+				)
+				(justify left)
+			)
+		)
+		(pin "O9" input
 			(at 76.2 46.99 0)
 			(effects
@@
 			)
 		)
-		(pin "OUT_8" input
+		(pin "O8" input
 			(at 76.2 44.45 0)
 			(effects
@@
 			)
 		)
-		(pin "OUT_10" input
+		(pin "O10" input
 			(at 76.2 49.53 0)
 			(effects
@@
 			)
 		)
-		(pin "RTS" input
+		(pin "DE{slash}~{RE}" input
 			(at 76.2 69.85 0)
 			(effects
@@
 			)
 		)
-		(pin "RESET" input
-			(at 63.5 57.15 180)
+		(pin "~{RST}" input
+			(at 63.5 55.88 180)
 			(effects
 				(font
@@
 			(color 255 255 194 1.0000)
 		)
-		(property "Sheetname" "IN"
+		(property "Sheetname" "PERIPHERALS"
 			(at 88.9 56.4384 0)
 			(effects
@@
 			)
 		)
-		(property "Sheetfile" "in.kicad_sch"
+		(property "Sheetfile" "peripherals.kicad_sch"
 			(at 88.9 75.5146 0)
 			(effects
@@
 		)
 		(pin "GND" input
-			(at 99.06 74.93 270)
-			(effects
-				(font
-					(size 1.27 1.27)
-				)
-				(justify left)
-			)
-		)
-		(pin "RXD" input
+			(at 95.25 74.93 270)
+			(effects
+				(font
+					(size 1.27 1.27)
+				)
+				(justify left)
+			)
+		)
+		(pin "RX" input
 			(at 88.9 67.31 180)
 			(effects
@@
 			)
 		)
-		(pin "TXD" input
+		(pin "TX" input
 			(at 88.9 64.77 180)
 			(effects
@@
 			)
 		)
-		(pin "TX_EN" input
+		(pin "DE" input
 			(at 88.9 69.85 180)
 			(effects
@@
 			)
 		)
-		(pin "~{RX_EN}" input
+		(pin "~{RE}" input
 			(at 88.9 72.39 180)
 			(effects

Commit message: feat
Parts:
- added J1: Screw_Terminal_01x04, symbol Connector:Screw_Terminal_01x04
- added J2, J3: Screw_Terminal_01x12, symbol Connector:Screw_Terminal_01x12
- renumbered J1 to J4
Connections:
- net +24V: now also J1.1 (Pin_1)
- net +5V: now also J1.4 (Pin_4)
- net GND: now also J1.2 (Pin_2), J1.3 (Pin_3)
- net OUT/L1: now also J2.1 (Pin_1)
- net OUT/L10: now also J2.10 (Pin_10)
- net OUT/L2: now also J2.2 (Pin_2)
- net OUT/L3: now also J2.3 (Pin_3)
- net OUT/L4: now also J2.4 (Pin_4)
- net OUT/L5: now also J2.5 (Pin_5)
- net OUT/L6: now also J2.6 (Pin_6)
- net OUT/L7: now also J2.7 (Pin_7)
- net OUT/L8: now also J2.8 (Pin_8)
- net OUT/L9: now also J2.9 (Pin_9)
- new net OUT/K1_COM: J3.1 (Pin_1)
- new net OUT/K1_NO: J3.2 (Pin_2)
- new net OUT/K2_COM: J3.3 (Pin_3)
- new net OUT/K2_NO: J3.4 (Pin_4)
- new net OUT/K3_COM: J3.5 (Pin_5)
- new net OUT/K3_NO: J3.6 (Pin_6)
- new net OUT/K4_COM: J3.7 (Pin_7)
- new net OUT/K4_NO: J3.8 (Pin_8)
- new net OUT/K5_COM: J3.9 (Pin_9)
- new net OUT/K5_NO: J3.10 (Pin_10)
- new net OUT/K6_COM: J3.11 (Pin_11)
- new net OUT/K6_NO: J3.12 (Pin_12)
- new net OUT/L11: J2.11 (Pin_11)
- new net OUT/L12: J2.12 (Pin_12)
Other:
- sheet MCU ports: added O11, O12, O13, O14, O15, O16, O17, O18; removed ~{RST}
- sheet OUT ports: added 5V, K1_COM, K1_NO, K2_COM, K2_NO, K3_COM, K3_NO, K4_COM, K4_NO, K5_COM, K5_NO, K6_COM, K6_NO, L11, L12, O11, O12, O13, O14, O15, O16, O17, O18; removed none
- note added: "NOTE: Predisporre ventola di raffreddamento e termocoppie Mettere fusibili Controllare pinout relay e opto"
- note removed: "NOTE: Chiedere se predisporre anche uscite per relay Predisporre ventola di raffreddamento e termocoppie Mettere fusibili Aggiungere altre zone con MOSFET (minimo 12)"
- moved on the sheet: J4, JP1

Commit message: !feat
Parts:
- removed J1: Screw_Terminal_01x04, symbol Connector:Screw_Terminal_01x04
- added J1, J2: Screw_Terminal_01x02, symbol Connector:Screw_Terminal_01x02
- renumbered J2 to J3, J3 to J4, J4 to J5
Connections:
- net +24V: now also J1.1 (Pin_1)
- net +5V: now also J2.1 (Pin_1)
- net GND: now also J1.2 (Pin_2), J2.2 (Pin_2)
- net OUT/K6_COM renamed AC_L
- net OUT/K6_NO renamed AC_N
Other:
- added sheet HOMEMONITOR (untitled.kicad_sch)
- added sheet PROTECTIONS (protections.kicad_sch)
- sheet MCU ports: added 3.3V, AC_I, AC_V, FAN, TEMP; removed O18
- sheet OUT ports: added none; removed K6_COM, K6_NO, O18
- sheet PERIPHERALS ports: added 24V, FAN; removed none
- note added: "NOTE: Fare footprint per trasformatore e pinsa amperometrica Mettere cicalino (attaccare ad un pin non strapping)"
- note removed: "NOTE: Predisporre ventola di raffreddamento e termocoppie Mettere fusibili Controllare pinout relay e opto"
- moved on the sheet: J3, J4, J5, JP1

Commit message: feat
Parts:
- added J5: Screw_Terminal_01x06, Connector_Phoenix_MC_D1.4mm:PhoenixContact_MCV_1,5_6-G-3.81_1x06_P3.81mm_D1.4mm_Vertical, symbol Connector:Screw_Terminal_01x06
- added J6, J7: Conn_01x03_Pin, Connector:FanPinHeader_1x03_P2.54mm_Vertical, symbol Connector:Conn_01x03_Pin
- added J8: AudioJack4, symbol Connector_Audio:AudioJack4
- J1, J2: footprint (none) -> Connector_Phoenix_MC_D1.4mm:PhoenixContact_MCV_1,5_2-G-3.81_1x02_P3.81mm_D1.4mm_Vertical
- J3, J4: footprint (none) -> Connector_Phoenix_MC_D1.4mm:PhoenixContact_MCV_1,5_12-G-3.81_1x12_P3.81mm_D1.4mm_Vertical
- renumbered J5 to J9
Connections:
- net OUT/K5_COM: no longer names the net of J4.9 (Pin_9)
- net OUT/K5_NO: no longer names the net of J4.10 (Pin_10)
- new net AC_I_IN_1: J8.1, J8.4
- new net AC_I_IN_2: J8.3
- new net PERIPHERALS/BUZZER+: J5.4 (Pin_4)
- new net PERIPHERALS/BUZZER-: J5.3 (Pin_3)
- new net PERIPHERALS/BUZZER_EN_1: J5.1 (Pin_1)
- new net PERIPHERALS/BUZZER_EN_2: J5.2 (Pin_2)
- new net PERIPHERALS/FAN+: J6.2 (Pin_2), J7.2 (Pin_2)
- new net PERIPHERALS/FAN-: J6.1 (Pin_1), J7.1 (Pin_1)
- new net PERIPHERALS/LED+: J5.6 (Pin_6)
- new net PERIPHERALS/LED-: J5.5 (Pin_5)
- no-connect marks 2 -> 5
Other:
- sheet HOMEMONITOR ports: added AC_I_IN_1, AC_I_IN_2; removed none
- sheet MCU ports: added ALARM; removed O17
- sheet OUT ports: added none; removed K5_COM, K5_NO, O17
- sheet PERIPHERALS ports: added ALARM, BUZZER+, BUZZER-, BUZZER_EN_1, BUZZER_EN_2, FAN+, FAN-, LED+, LED-; removed none
- note added: "NOTE: Fare footprint per trasformatore, pinsa amperometrica"
- note removed: "NOTE: Fare footprint per trasformatore e pinsa amperometrica Mettere cicalino (attaccare ad un pin non strapping)"
- moved on the sheet: J3, J4, J9, JP1

Commit message: !feat
Parts:
- removed J1, J2: Screw_Terminal_01x02, Connector_Phoenix_MC_D1.4mm:PhoenixContact_MCV_1,5_2-G-3.81_1x02_P3.81mm_D1.4mm_Vertical, symbol Connector:Screw_Terminal_01x02
- removed J4: Screw_Terminal_01x12, Connector_Phoenix_MC_D1.4mm:PhoenixContact_MCV_1,5_12-G-3.81_1x12_P3.81mm_D1.4mm_Vertical, symbol Connector:Screw_Terminal_01x12
- removed J5: Screw_Terminal_01x06, Connector_Phoenix_MC_D1.4mm:PhoenixContact_MCV_1,5_6-G-3.81_1x06_P3.81mm_D1.4mm_Vertical, symbol Connector:Screw_Terminal_01x06
- added F1: T30A 250V, Fuse:Fuseholder_Clip-6.3x32mm_Littelfuse_102_Inline_P34.21x7.62mm_D2.54mm_Horizontal, symbol Device:Fuse
- added J2, J3, J5: Screw_Terminal_01x08, Connector_Phoenix_MC_D1.4mm:PhoenixContact_MCV_1,5_8-G-3.81_1x08_P3.81mm_D1.4mm_Vertical, symbol Connector:Screw_Terminal_01x08
- J4: renamed from J8; footprint (none) -> HomeMonitor:SCT013
- renumbered J3 to J1, J9 to J6, J6 to J7, J7 to J8
Connections:
- net +24V: now also J5.4 (Pin_4)
- net +3.3V: now also J5.8 (Pin_8)
- net +5V: now also J5.6 (Pin_6)
- net AC_I_IN_1: now also J4.R2, J4.S; no longer J4.1, J4.4
- net AC_I_IN_2: now also J4.T; no longer J4.3
- net AC_L: now also J5.1 (Pin_1)
- net AC_N: now also J5.2 (Pin_2)
- net GND: now also F1.2, J3.8 (Pin_8)
- net OUT/K1_COM: now also J2.1 (Pin_1)
- net OUT/K1_NO: now also J2.2 (Pin_2)
- net OUT/K2_COM: now also J2.3 (Pin_3)
- net OUT/K2_NO: now also J2.4 (Pin_4)
- net OUT/K3_COM: now also J2.5 (Pin_5)
- net OUT/K3_NO: now also J2.6 (Pin_6)
- net OUT/K4_COM: now also J2.7 (Pin_7)
- net OUT/K4_NO: now also J2.8 (Pin_8)
- net PERIPHERALS/BUZZER+: now also J3.4 (Pin_4)
- net PERIPHERALS/BUZZER-: now also J3.3 (Pin_3)
- net PERIPHERALS/BUZZER_EN_1: now also J3.1 (Pin_1)
- net PERIPHERALS/BUZZER_EN_2: now also J3.2 (Pin_2)
- net PERIPHERALS/LED+: now also J3.6 (Pin_6)
- net PERIPHERALS/LED-: now also J3.5 (Pin_5)
- new net: F1.1, J5.3 (Pin_3), J5.5 (Pin_5), J5.7 (Pin_7)
- new net ~{RESET}: J3.7 (Pin_7)
Other:
- sheet MCU ports: added ~{RESET}; removed none
- note removed: "NOTE: Fare footprint per trasformatore, pinsa amperometrica"
- moved on the sheet: J4, J6, J7, J8
