File: hardware/schematics/control_unit/control_unit.kicad_pcb (KiCad board)
At the start: 2 copper layers, 129 parts, among them J1 Screw_Terminal_01x12, J2 Screw_Terminal_01x08, J3 Screw_Terminal_01x08, J4 AudioJack4, J5 Screw_Terminal_01x08, J6 6P6C, J7 Conn_01x03_Pin, J8 Conn_01x03_Pin, K1 Relay_SPDT, K2 Relay_SPDT, K3 Relay_SPDT, K4 Relay_SPDT, Q1 2N7000, Q10 IRFZ44N, Q11 IRFZ44N, Q12 IRFZ44N, Q13 IRFZ44N, Q14 IRFZ44N, Q15 IRFZ44N, Q16 IRFZ44N, Q17 IRFZ44N, Q18 2N7000, Q2 2N7000, Q3 IRFZ44N, Q4 IRFZ44N, Q5 IRFZ44N, Q6 2N7000, Q7 2N7000, Q8 IRFZ44N, Q9 IRFZ44N, T1 Transformer_1P_1S, U1 PC817, U10 PC817, U11 PC817, U12 PC817, U13 PC817, U14 MAX487E, U15 ESP-WROOM-32, U16 LM2596T-ADJ, U17 LM35-D, U18 LM324, U2 PC817, U3 PC817, U4 PC817, U5 PC817, U6 PC817, U7 PC817, U8 PC817, U9 PC817

Commit message: !feat
Parts:
- added G***: LOGO, LOGO, F.Cu at (132.3, 112.0)
- added H1: MountingHole, MountingHole:MountingHole_4.5mm_Pad_TopBottom, F.Cu at (104.4, 79.5)
- added H2: MountingHole, MountingHole:MountingHole_4.5mm_Pad_TopBottom, F.Cu at (220.5, 68.8)
- added H3: MountingHole, MountingHole:MountingHole_4.5mm_Pad_TopBottom, F.Cu at (87.6, 124.7)
- added H4: MountingHole, MountingHole:MountingHole_4.5mm_Pad_TopBottom, F.Cu at (203.7, 131.6)
- moved J7 225.6 mm to (221.3, 121.4), turned to 90 degrees
- moved R57 207.8 mm to (83.6, 116.3)
- moved C7 203.7 mm to (79.8, 116.3), turned to 180 degrees
- moved R55 198.5 mm to (105.4, 128.5)
- moved R59 198.0 mm to (105.4, 143.8)
- moved R56 198.0 mm to (105.4, 131.6)
- moved R60 197.1 mm to (94.0, 125.5)
- moved R58 192.2 mm to (113.0, 140.7), turned to 180 degrees
- moved R61 185.1 mm to (105.4, 125.5)
- moved R47 185.0 mm to (91.4, 135.6), turned to -90 degrees
- moved J6 184.0 mm to (86.9, 139.7), turned to -90 degrees
- moved R52 179.8 mm to (92.2, 109.5)
- moved U14 176.7 mm to (102.6, 140.7), turned to 180 degrees
- moved JP1 175.7 mm to (101.3, 143.6)
- moved U17 171.9 mm to (100.8, 104.0)
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Connections:
- JP1 pad 1: GND -> /MCU/DE/~{RE}
- JP1 pad 3: /MCU/DE/~{RE} -> GND
- R44 pad 1: /MCU/RX -> Net-(U14-RO)
- R44 pad 2: Net-(U14-RO) -> /MCU/RX
- R45 pad 1: GND -> /MCU/RX
- R45 pad 2: /MCU/RX -> GND
- R48 pad 1: /PERIPHERALS/BUZZER_EN_2 -> /PERIPHERALS/LED-
- R48 pad 2: /PERIPHERALS/LED- -> /PERIPHERALS/BUZZER_EN_2
- R51 pad 1: +5V -> Net-(D8-A)
- R51 pad 2: Net-(D8-A) -> +5V
- R53 pad 1: GND -> Net-(U18A--)
- R53 pad 2: Net-(U18A--) -> GND
- R55 pad 1: +3.3V -> /AC_I_IN_1
- R55 pad 2: /AC_I_IN_1 -> +3.3V
- R60 pad 1: Net-(U18C--) -> /HOMEMONITOR/I
- R60 pad 2: /HOMEMONITOR/I -> Net-(U18C--)
Other:
- board outline added: 151.3 x 95.4 mm
- board text added: "JLCJLCJLCJLC"
- board text added: "~{ECHO}/ECHO"
