File: hardware/schematics/control_unit/untitled.kicad_sch (KiCad schematic)
At the start: 8 parts, among them T1 Transformer_1P_1S

Commit message: feat
Parts:
- removed L2: L, symbol Device:L
- added R60, R61: 10k, Resistor_THT:R_Axial_DIN0207_L6.3mm_D2.5mm_P7.62mm_Horizontal, symbol Device:R
- added U18: LM324, Package_DIP:DIP-14_W7.62mm_Socket, symbol Amplifier_Operational:LM324
- C7: footprint (none) -> Capacitor_THT:CP_Radial_D4.0mm_P2.00mm
- R55: renamed from R52; footprint (none) -> Resistor_THT:R_Axial_DIN0207_L6.3mm_D2.5mm_P7.62mm_Horizontal
- R56: renamed from R53; footprint (none) -> Resistor_THT:R_Axial_DIN0207_L6.3mm_D2.5mm_P7.62mm_Horizontal
- R57: renamed from R54; footprint (none) -> Resistor_THT:R_Axial_DIN0207_L6.3mm_D2.5mm_P7.62mm_Horizontal
- R58: renamed from R55; footprint (none) -> Resistor_THT:R_Axial_DIN0207_L6.3mm_D2.5mm_P7.62mm_Horizontal
- R59: renamed from R56; footprint (none) -> Resistor_THT:R_Axial_DIN0207_L6.3mm_D2.5mm_P7.62mm_Horizontal
Connections:
- net I: now also R60.2, U18.8; no longer R57.2
- net V: now also R61.2, U18.14; no longer R58.2, R59.1
- net 1.65V renamed AC_I_IN_1
- new net: R61.1, U18.13 (-)
- new net: R60.1, U18.9 (-)
- new net: R58.2, R59.1, U18.12 (+)
- new net AC_I_IN_2: R57.2, U18.10 (+)
Other:
- moved on the sheet: R57

Commit message: !feat
Parts:
- T1: footprint (none) -> HomeMonitor:Transformer
Connections:
- net AC_I_IN_1: now also T1.4 (SB); no longer T1.3 (SA)
- net AC_L: now also T1.2 (AB); no longer T1.1 (AA)
- net AC_N: now also T1.1 (AA); no longer T1.2 (AB)
- net at R58.1: now also T1.3 (SA); no longer T1.4 (SB)
Changed lines of the file:
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@@
 		(lib_id "Device:Transformer_1P_1S")
 		(at 144.78 100.33 0)
+		(mirror x)
 		(unit 1)
 		(exclude_from_sim no)
@@
 		)
 		(property "Value" "Transformer_1P_1S"
-			(at 144.7927 92.71 0)
+			(at 144.7927 107.95 0)
 			(effects
 				(font
@@
 			)
 		)
-		(property "Footprint" ""
+		(property "Footprint" "HomeMonitor:Transformer"
 			(at 144.78 100.33 0)
 			(effects

Commit message: !feat
Connections:
- net 3.3V: now also R55.2; no longer R55.1
- net AC_I_IN_1: now also R55.1; no longer R55.2
- net I: now also R60.1; no longer R60.2
- net at U18.9 (-): now also R60.2; no longer R60.1
Other:
- moved on the sheet: R55, R60
Changed lines of the file:
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@@
 	(symbol
 		(lib_id "Device:R")
-		(at 190.5 87.63 90)
-		(mirror x)
+		(at 190.5 87.63 270)
 		(unit 1)
 		(exclude_from_sim no)
@@
 	(symbol
 		(lib_id "Device:R")
-		(at 101.6 86.36 0)
+		(at 101.6 86.36 180)
 		(unit 1)
 		(exclude_from_sim no)
@@
 					(size 1.27 1.27)
 				)
-				(justify left)
+				(justify right)
 			)
 		)
@@
 					(size 1.27 1.27)
 				)
-				(justify left)
-			)
-		)
-		(property "Footprint" "Resistor_THT:R_Axial_DIN0207_L6.3mm_D2.5mm_P7.62mm_Horizontal"
-			(at 99.822 86.36 90)
-			(effects
-				(font
+				(justify right)
+			)
+		)
+		(property "Footprint" "Resistor_THT:R_Axial_DIN0207_L6.3mm_D2.5mm_P7.62mm_Horizontal"
+			(at 103.378 86.36 90)
+			(effects
+				(font
