File: hardware/schematics/control_unit/out.kicad_sch (KiCad schematic)
At the start: 50 parts, among them Q1 IRFZ44N, Q10 IRFZ44N, Q2 IRFZ44N, Q3 IRFZ44N, Q4 IRFZ44N, Q5 IRFZ44N, Q6 IRFZ44N, Q7 IRFZ44N, Q8 IRFZ44N, Q9 IRFZ44N, U10 PC817, U11 PC817, U12 PC817, U13 PC817, U4 PC817, U5 PC817, U6 PC817, U7 PC817, U8 PC817, U9 PC817

Commit message: chore
Parts:
- renumbered Q7 to Q1, Q3 to Q10, Q8 to Q2, Q9 to Q3, Q10 to Q4, Q4 to Q5, Q5 to Q6, Q6 to Q7, Q1 to Q8, Q2 to Q9, R23 to R1, R31 to R10, R33 to R11, R34 to R12, R14 to R13, R15 to R14, R16 to R15, R17 to R16, R18 to R17, R19 to R18, R20 to R19, R24 to R2, R21 to R20, R22 to R21, R5 to R22, R8 to R23, R11 to R24, R7 to R25, R6 to R26, R9 to R27, R10 to R28, R12 to R29, R25 to R3, R13 to R30, R32 to R4, R26 to R5, R27 to R6, R28 to R7, R29 to R8, R30 to R9, U10 to U1, U6 to U10, U11 to U2, U12 to U3, U13 to U4, U7 to U5, U8 to U6, U9 to U7, U4 to U8, U5 to U9

Commit message: !refactor
Connections:
- net LED_1 renamed L1
- net LED_10 renamed L10
- net LED_2 renamed L2
- net LED_3 renamed L3
- net LED_4 renamed L4
- net LED_5 renamed L5
- net LED_6 renamed L6
- net LED_7 renamed L7
- net LED_8 renamed L8
- net LED_9 renamed L9
- net OUT_1 renamed O1
- net OUT_10 renamed O10
- net OUT_2 renamed O2
- net OUT_3 renamed O3
- net OUT_4 renamed O4
- net OUT_5 renamed O5
- net OUT_6 renamed O6
- net OUT_7 renamed O7
- net OUT_8 renamed O8
- net OUT_9 renamed O9
Changed lines of the file:
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@@
 		)
 	)
-	(hierarchical_label "OUT_9"
+	(hierarchical_label "O9"
 		(shape input)
 		(at 91.44 111.76 180)
@@
 		)
 	)
-	(hierarchical_label "OUT_1"
+	(hierarchical_label "O1"
 		(shape input)
 		(at 218.44 35.56 180)
@@
 		)
 	)
-	(hierarchical_label "LED_9"
+	(hierarchical_label "L9"
 		(shape input)
 		(at 128.27 110.49 0)
@@
 		)
 	)
-	(hierarchical_label "OUT_10"
+	(hierarchical_label "O10"
 		(shape input)
 		(at 91.44 149.86 180)
@@
 		)
 	)
-	(hierarchical_label "OUT_5"
+	(hierarchical_label "O5"
 		(shape input)
 		(at 154.94 73.66 180)
@@
 		)
 	)
-	(hierarchical_label "OUT_7"
+	(hierarchical_label "O7"
 		(shape input)
 		(at 91.44 35.56 180)
@@
 		)
 	)
-	(hierarchical_label "LED_4"
+	(hierarchical_label "L4"
 		(shape input)
 		(at 191.77 34.29 0)
@@
 		)
 	)
-	(hierarchical_label "LED_8"
+	(hierarchical_label "L8"
 		(shape input)
 		(at 128.27 72.39 0)
@@
 		)
 	)
-	(hierarchical_label "LED_6"
+	(hierarchical_label "L6"
 		(shape input)
 		(at 191.77 110.49 0)
@@
 		)
 	)
-	(hierarchical_label "LED_2"
+	(hierarchical_label "L2"
 		(shape input)
 		(at 255.27 72.39 0)
@@
 		)
 	)
-	(hierarchical_label "LED_3"
+	(hierarchical_label "L3"
 		(shape input)
 		(at 255.27 110.49 0)
@@
 		)
 	)
-	(hierarchical_label "OUT_8"
+	(hierarchical_label "O8"
 		(shape input)
 		(at 91.44 73.66 180)
@@
 		)
 	)
-	(hierarchical_label "LED_1"
+	(hierarchical_label "L1"
 		(shape input)
 		(at 255.27 34.29 0)
@@
 		)
 	)
-	(hierarchical_label "OUT_2"
+	(hierarchical_label "O2"
 		(shape input)
 		(at 218.44 73.66 180)
@@
 		)
 	)
-	(hierarchical_label "LED_7"
+	(hierarchical_label "L7"
 		(shape input)
 		(at 128.27 34.29 0)
@@
 		)
 	)
-	(hierarchical_label "OUT_6"
+	(hierarchical_label "O6"
 		(shape input)
 		(at 154.94 111.76 180)
@@
 		)
 	)
-	(hierarchical_label "OUT_4"
+	(hierarchical_label "O4"
 		(shape input)
 		(at 154.94 35.56 180)
@@
 		)
 	)
-	(hierarchical_label "LED_10"
+	(hierarchical_label "L10"
 		(shape input)
 		(at 128.27 148.59 0)
@@
 		)
 	)
-	(hierarchical_label "LED_5"
+	(hierarchical_label "L5"
 		(shape input)
 		(at 191.77 72.39 0)
@@
 		)
 	)
-	(hierarchical_label "OUT_3"
+	(hierarchical_label "O3"
 		(shape input)
 		(at 218.44 111.76 180)

Commit message: feat
Parts:
- removed Q10, Q4, Q8, Q9: IRFZ44N, Package_TO_SOT_THT:TO-220-3_Vertical, symbol Transistor_FET:IRF540N
- removed R11, R12: 1k, symbol Device:R
- removed R22: R, symbol Device:R
- removed U4: PC817, Package_DIP:DIP-4_W7.62mm, symbol Isolator:PC817
- added D1, D2, D3, D4, D5, D6: 1N4007, Diode_THT:D_DO-41_SOD81_P2.54mm_Vertical_KathodeUp, symbol Diode:1N4007
- added JP10, JP11, JP12, JP13, JP16, JP17, JP2, JP20, JP21, JP22, JP23, JP24, JP25, JP3, JP4, JP5, JP6, JP9: SolderJumper_2_Open, symbol Jumper:SolderJumper_2_Open
- added JP14, JP15, JP18, JP19, JP7, JP8: SolderJumper_3_Open, Jumper:SolderJumper-3_P1.3mm_Open_Pad1.0x1.5mm, symbol Jumper:SolderJumper_3_Open
- added K1, K2, K3, K4, K5, K6: Relay_SPDT, Relay_THT:Relay_SPDT_Omron-G5LE-1, symbol Relay:Relay_SPDT
- added Q1, Q11, Q12, Q2, Q6, Q7: 2N7000, Package_TO_SOT_THT:TO-92_Inline, symbol Transistor_FET:2N7000
- added Q13, Q14, Q15, Q16, Q17, Q18: IRFZ44N, Package_TO_SOT_THT:TO-220-3_Vertical, symbol Transistor_FET:IRF540N
- added R15, R16, R34, R35, R36, R5: R, symbol Device:R
- added R31, R32, R33, R37, R38, R39, R40, R41, R42: 1k, symbol Device:R
- added U11, U12, U7: PC817, Package_DIP:DIP-4_W7.62mm, symbol Isolator:PC817
- R25, R26, R27: value 1k -> R
- renumbered Q7 to Q10, Q1 to Q3, Q2 to Q4, Q3 to Q5, Q5 to Q8, Q6 to Q9, R9 to R10, R10 to R11, R13 to R12, R14 to R13, R15 to R14, R16 to R17, R17 to R18, R18 to R19, R19 to R20, R20 to R21, R21 to R22, R5 to R6, R6 to R7, R7 to R8, R8 to R9, U5 to U4, U6 to U5, U7 to U6
Connections:
- net 24V: now also R28.1, R30.1, JP11.2 (B), JP12.2 (B), JP13.2 (B), JP14.1 (A), JP15.1 (A), JP18.1 (A), JP19.1 (A), JP2.2 (B), JP20.2 (B), JP21.2 (B), JP22.2 (B), JP23.2 (B), JP24.2 (B), JP25.2 (B), JP3.2 (B), JP4.2 (B), JP7.1 (A), JP8.1 (A), R32.1, R37.1, R39.1, R41.1; no longer R25.1, R27.1, R29.1
- net GND: now also R29.2, Q1.1 (S), Q11.1 (S), Q12.1 (S), Q13.3 (S), Q14.3 (S), Q15.3 (S), Q16.3 (S), Q17.3 (S), Q18.3 (S), Q2.1 (S), Q6.1 (S), Q7.1 (S), R31.2, R33.2, R38.2, R40.2, R42.2, U11.2, U12.2, U7.2; no longer R26.2, R28.2, R30.2
- net L1: now also Q3.2 (D)
- net L10: now also Q16.2 (D)
- net L2: now also Q4.2 (D)
- net L3: now also Q5.2 (D)
- net L7: now also Q13.2 (D); no longer Q3.2 (D)
- net L8: now also Q14.2 (D); no longer Q4.2 (D)
- net L9: now also Q15.2 (D); no longer Q5.2 (D)
- net O1: now also R1.1
- net O10: now also R34.1; no longer R4.1
- net O2: now also R2.1; no longer R23.1
- net O3: now also R3.1; no longer R24.1
- net O7: now also R23.1; no longer R1.1
- net O8: now also R24.1; no longer R2.1
- net O9: now also R25.1; no longer R3.1
- net at R8.2, U2.4: now also JP3.1 (A)
- net at R10.2, U3.4: now also JP4.1 (A)
- net at R4.2: now also JP5.1 (A), JP7.2 (C)
- net at U10.1: now also R34.2; no longer R24.2
- net at U10.3: now also Q16.1 (G), R38.1; no longer R30.1
- net at U10.4: now also JP23.1 (A), R37.2; no longer R29.2
- net at U9.3: now also Q15.1 (G), R33.1; no longer R28.1
- net at R17.2, U4.4: now also JP11.1 (A)
- net at R21.2, U6.4: now also JP13.1 (A)
- net at R26.1: now also D5.1 (K), JP16.2 (B), K5.5; no longer U8.3
- net at R19.2, U5.4: now also JP12.1 (A)
- net at U8.1: now also R24.2
- net at R6.2, U1.4: now also JP2.1 (A)
- net at R25.2: now also U9.1; no longer U8.4
- net at R23.2: now also U7.1; no longer U9.1
- net at R27.2: now also JP17.1 (A), JP19.2 (C); no longer U9.4
- new net: D3.2 (A), K3.2, Q6.3 (D)
- new net: D3.1 (K), JP9.2 (B), K3.5, R15.1
- new net: JP14.2 (C), JP9.1 (A), R15.2
- new net: Q17.1 (G), R40.1, U11.3
- new net: D6.2 (A), K6.2, Q12.3 (D)
- new net: D1.1 (K), JP5.2 (B), K1.5, R4.1
- new net: D1.2 (A), K1.2, Q1.3 (D)
- new net: JP16.1 (A), JP18.2 (C), R26.2
- new net: D2.2 (A), K2.2, Q2.3 (D)
- new net: D2.1 (K), JP6.2 (B), K2.5, R5.1
- new net: JP22.1 (A), R32.2, U9.4
- new net: JP6.1 (A), JP8.2 (C), R5.2
- new net: R35.2, U11.1
- new net: JP24.1 (A), R39.2, U11.4
- new net: D4.1 (K), JP10.2 (B), K4.5, R16.1
- new net: JP10.1 (A), JP15.2 (C), R16.2
- new net: D4.2 (A), K4.2, Q7.3 (D)
- new net: D6.1 (K), JP17.2 (B), K6.5, R27.1
- new net: JP20.1 (A), R28.2, U7.4
- new net: Q13.1 (G), R29.1, U7.3
- new net: JP25.1 (A), R41.2, U12.4
- new net: JP21.1 (A), R30.2, U8.4
- new net: D5.2 (A), K5.2, Q11.3 (D)
- new net: Q14.1 (G), R31.1, U8.3
- new net: Q18.1 (G), R42.1, U12.3
- new net: R36.2, U12.1
- new net 5V: JP14.3 (B), JP15.3 (B), JP18.3 (B), JP19.3 (B), JP7.3 (B), JP8.3 (B)
- new net K1_COM: K1.1
- new net K1_NO: K1.3
- new net K2_COM: K2.1
- new net K2_NO: K2.3
- new net K3_COM: K3.1
- new net K3_NO: K3.3
- new net K4_COM: K4.1
- new net K4_NO: K4.3
- new net K5_COM: K5.1
- new net K5_NO: K5.3
- new net K6_COM: K6.1
- new net K6_NO: K6.3
- new net L11: Q17.2 (D)
- new net L12: Q18.2 (D)
- new net O11: Q1.2 (G)
- new net O12: Q2.2 (G)
- new net O13: Q6.2 (G)
- new net O14: Q7.2 (G)
- new net O15: Q11.2 (G)
- new net O16: Q12.2 (G)
- new net O17: R35.1
- new net O18: R36.1
- no-connect marks 0 -> 6
Other:
- moved on the sheet: Q10, Q3, Q4, Q5, Q8, Q9, R1, R10, R11, R12, R13, R14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

Commit message: !feat
Parts:
- removed D6: 1N4007, Diode_THT:D_DO-41_SOD81_P2.54mm_Vertical_KathodeUp, symbol Diode:1N4007
- removed JP10, JP16, JP17, JP5, JP6, JP9: SolderJumper_2_Open, symbol Jumper:SolderJumper_2_Open
- removed JP15, JP18, JP19, JP7, JP8: SolderJumper_3_Open, Jumper:SolderJumper-3_P1.3mm_Open_Pad1.0x1.5mm, symbol Jumper:SolderJumper_3_Open
- removed K6: Relay_SPDT, Relay_THT:Relay_SPDT_Omron-G5LE-1, symbol Relay:Relay_SPDT
- removed Q12: 2N7000, Package_TO_SOT_THT:TO-92_Inline, symbol Transistor_FET:2N7000
- removed R15, R16, R27, R4, R5: R, symbol Device:R
- added R1, R12, R13, R2: 10k, symbol Device:R
- JP14: value SolderJumper_3_Open -> (none)
- R26: value R -> 10k
- renumbered JP22 to JP10, JP23 to JP11, JP24 to JP12, JP25 to JP13, JP11 to JP5, JP12 to JP6, JP13 to JP7, JP20 to JP8, JP21 to JP9, Q13 to Q12, Q14 to Q13, Q15 to Q14, Q16 to Q15, Q17 to Q16, Q18 to Q17, R12 to R14, R13 to R15, R14 to R16, R28 to R27, R29 to R28, R30 to R29, R1 to R3, R31 to R30, R32 to R31, R33 to R32, R34 to R33, R35 to R34, R36 to R35, R37 to R36, R38 to R37, R39 to R38, R40 to R39, R2 to R4, R41 to R40, R42 to R41, R3 to R5
Connections:
- net O18 is gone; now on net O12: R35.1
- net 24V: no longer JP14.1 (A)
- net 5V: now also D1.1 (K), D2.1 (K), D3.1 (K), D4.1 (K), D5.1 (K), K1.5, K2.5, K3.5, K4.5, K5.5; no longer JP14.3 (B)
- net GND: now also R26.2, R1.2, R12.2, R13.2, R2.2
- net O11: now also R34.1; no longer Q1.2 (G)
- net O12: no longer Q2.2 (G)
- net O13: now also Q1.2 (G), R1.1; no longer Q6.2 (G)
- net O14: now also Q2.2 (G), R2.1; no longer Q7.2 (G)
- net O15: now also Q6.2 (G), R12.1; no longer Q11.2 (G)
- net O16: now also Q7.2 (G), R13.1
- net O17: now also Q11.2 (G), R26.1; no longer R34.1
- no-connect marks 6 -> 5
Other:
- moved on the sheet: D1, D2, D3, D4, D5, K1, K2, K3, K4, K5, Q1, Q11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

Commit message: feat
Parts:
- removed D5: 1N4007, Diode_THT:D_DO-41_SOD81_P2.54mm_Vertical_KathodeUp, symbol Diode:1N4007
- removed JP10, JP11, JP12, JP13, JP2, JP3, JP4, JP5, JP6, JP7, JP8, JP9: SolderJumper_2_Open, symbol Jumper:SolderJumper_2_Open
- removed JP14: (no value), Jumper:SolderJumper-3_P1.3mm_Open_Pad1.0x1.5mm, symbol Jumper:SolderJumper_3_Open
- removed K5: Relay_SPDT, Relay_THT:Relay_SPDT_Omron-G5LE-1, symbol Relay:Relay_SPDT
- removed Q11: 2N7000, Package_TO_SOT_THT:TO-92_Inline, symbol Transistor_FET:2N7000
- removed R26: 10k, symbol Device:R
- R1, R10, R11, R12, R13, R14, R15, R16, R17, R18, R19, R2, R20, R21, R22, R23, R24, R25, R3, R4, R5, R6, R7, R8, R9: footprint (none) -> Resistor_THT:R_Axial_DIN0207_L6.3mm_D2.5mm_P7.62mm_Horizontal
- R26: renamed from R27; footprint (none) -> Resistor_THT:R_Axial_DIN0207_L6.3mm_D2.5mm_P7.62mm_Horizontal
- R27: renamed from R28; footprint (none) -> Resistor_THT:R_Axial_DIN0207_L6.3mm_D2.5mm_P7.62mm_Horizontal
- R28: renamed from R29; footprint (none) -> Resistor_THT:R_Axial_DIN0207_L6.3mm_D2.5mm_P7.62mm_Horizontal
- R29: renamed from R30; footprint (none) -> Resistor_THT:R_Axial_DIN0207_L6.3mm_D2.5mm_P7.62mm_Horizontal
- R30: renamed from R31; footprint (none) -> Resistor_THT:R_Axial_DIN0207_L6.3mm_D2.5mm_P7.62mm_Horizontal
- R31: renamed from R32; footprint (none) -> Resistor_THT:R_Axial_DIN0207_L6.3mm_D2.5mm_P7.62mm_Horizontal
- R32: renamed from R33; footprint (none) -> Resistor_THT:R_Axial_DIN0207_L6.3mm_D2.5mm_P7.62mm_Horizontal
- R33: renamed from R34; footprint (none) -> Resistor_THT:R_Axial_DIN0207_L6.3mm_D2.5mm_P7.62mm_Horizontal
- R34: renamed from R35; footprint (none) -> Resistor_THT:R_Axial_DIN0207_L6.3mm_D2.5mm_P7.62mm_Horizontal
- R35: renamed from R36; footprint (none) -> Resistor_THT:R_Axial_DIN0207_L6.3mm_D2.5mm_P7.62mm_Horizontal
- R36: renamed from R37; footprint (none) -> Resistor_THT:R_Axial_DIN0207_L6.3mm_D2.5mm_P7.62mm_Horizontal
- R37: renamed from R38; footprint (none) -> Resistor_THT:R_Axial_DIN0207_L6.3mm_D2.5mm_P7.62mm_Horizontal
- R38: renamed from R39; footprint (none) -> Resistor_THT:R_Axial_DIN0207_L6.3mm_D2.5mm_P7.62mm_Horizontal
- R39: renamed from R40; footprint (none) -> Resistor_THT:R_Axial_DIN0207_L6.3mm_D2.5mm_P7.62mm_Horizontal
- R40: renamed from R41; footprint (none) -> Resistor_THT:R_Axial_DIN0207_L6.3mm_D2.5mm_P7.62mm_Horizontal
- renumbered Q12 to Q11, Q13 to Q12, Q14 to Q13, Q15 to Q14, Q16 to Q15, Q17 to Q16
Connections:
- no-connect marks 5 -> 4

Commit message: !feat
Parts:
- D1, D2, D3, D4: footprint Diode_THT:D_DO-41_SOD81_P2.54mm_Vertical_KathodeUp -> Diode_THT:D_DO-41_SOD81_P7.62mm_Horizontal
Connections:
- net 24V: now also R10.2, R17.2, R19.2, R21.2, R26.2, R28.2, R30.2, R35.2, R37.2, R39.2, R6.2, R8.2; no longer R10.1, R17.1, R19.1, R21.1, R26.1, R28.1, R30.1, R35.1, R37.1, R39.1, R6.1, R8.1
- net GND: now also R1.1, R11.1, R12.1, R13.1, R18.1, R2.1, R20.1, R22.1, R27.1, R29.1, R31.1, R36.1, R38.1, R40.1, R7.1, R9.1; no longer R1.2, R11.2, R12.2, R13.2, R18.2, R2.2, R20.2, R22.2, R27.2, R29.2, R31.2, R36.2, R38.2, R40.2, R7.2, R9.2
- net O13: now also R1.2; no longer R1.1
- net O14: now also R2.2; no longer R2.1
- net O15: now also R12.2; no longer R12.1
- net O16: now also R13.2; no longer R13.1
- net at U2.4: now also R8.1; no longer R8.2
- net at Q9.1 (G), U5.3: now also R20.2; no longer R20.1
- net at Q15.1 (G), U11.3: now also R38.2; no longer R38.1
- net at U10.4: now also R35.1; no longer R35.2
- net at U3.4: now also R10.1; no longer R10.2
- net at Q5.1 (G), U3.3: now also R11.2; no longer R11.1
- net at U9.4: now also R30.1; no longer R30.2
- net at Q4.1 (G), U2.3: now also R9.2; no longer R9.1
- net at Q3.1 (G), U1.3: now also R7.2; no longer R7.1
- net at U11.4: now also R37.1; no longer R37.2
- net at U7.4: now also R26.1; no longer R26.2
- net at Q13.1 (G), U9.3: now also R31.2; no longer R31.1
- net at Q11.1 (G), U7.3: now also R27.2; no longer R27.1
- net at Q14.1 (G), U10.3: now also R36.2; no longer R36.1
- net at Q8.1 (G), U4.3: now also R18.2; no longer R18.1
- net at U4.4: now also R17.1; no longer R17.2
- net at Q10.1 (G), U6.3: now also R22.2; no longer R22.1
- net at U6.4: now also R21.1; no longer R21.2
- net at U5.4: now also R19.1; no longer R19.2
- net at U1.4: now also R6.1; no longer R6.2
- net at U8.4: now also R28.1; no longer R28.2
- net at Q12.1 (G), U8.3: now also R29.2; no longer R29.1
- net at Q16.1 (G), U12.3: now also R40.2; no longer R40.1
- net at U12.4: now also R39.1; no longer R39.2
Other:
- moved on the sheet: R1, R10, R11, R12, R13, R17, R18, R19, R2, R20, R21, R22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
