File: hardware/schematics/control_unit/peripherals.kicad_sch (KiCad schematic)
At the start: 4 parts, among them U11 MAX487E

Commit message: !refactor
Connections:
- net A: now also R33.1; no longer R33.2
- net B: now also R33.2; no longer R33.1
- net RXD renamed RX
- net TXD renamed TX
Other:
- moved on the sheet: R31, R32, R33

Commit message: feat
Parts:
- renumbered R31 to R43, R32 to R44, R33 to R45, U11 to U13
Changed lines of the file:
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@@
 		(dnp no)
 		(fields_autoplaced yes)
-		(property "Reference" "R33"
+		(property "Reference" "R45"
 			(at 156.21 81.2799 0)
 			(effects
@@
 			(project "control_unit"
 				(path "/95f83be4-8e7e-4d00-b795-d60cd8e47b85/8904da64-7973-4a3f-8dc5-f09a7326cd0e"
-					(reference "R33")
+					(reference "R45")
 					(unit 1)
 				)
@@
 		(on_board yes)
 		(dnp no)
-		(property "Reference" "R31"
+		(property "Reference" "R43"
 			(at 120.65 85.0899 0)
 			(effects
@@
 			(project "control_unit"
 				(path "/95f83be4-8e7e-4d00-b795-d60cd8e47b85/8904da64-7973-4a3f-8dc5-f09a7326cd0e"
-					(reference "R31")
+					(reference "R43")
 					(unit 1)
 				)
@@
 		(on_board yes)
 		(dnp no)
-		(property "Reference" "U11"
+		(property "Reference" "U13"
 			(at 141.986 69.85 0)
 			(effects
@@
 			(project "control_unit"
 				(path "/95f83be4-8e7e-4d00-b795-d60cd8e47b85/8904da64-7973-4a3f-8dc5-f09a7326cd0e"
-					(reference "U11")
+					(reference "U13")
 					(unit 1)
 				)
@@
 		(on_board yes)
 		(dnp no)
-		(property "Reference" "R32"
+		(property "Reference" "R44"
 			(at 120.65 95.2499 0)
 			(effects
@@
 			(project "control_unit"
 				(path "/95f83be4-8e7e-4d00-b795-d60cd8e47b85/8904da64-7973-4a3f-8dc5-f09a7326cd0e"
-					(reference "R32")
-					(unit 1)
-				)
+					(reference "R44")
+					(unit 1)
+				)

Commit message: !feat
Parts:
- added D6: 1N4007, Diode_THT:D_DO-41_SOD81_P2.54mm_Vertical_KathodeUp, symbol Diode:1N4007
- added M1: Fan, symbol Motor:Fan
- added Q18: 2N7000, Package_TO_SOT_THT:TO-92_Inline, symbol Transistor_FET:2N7000
- added R44: 10k, symbol Device:R
- renumbered R43 to R42, R44 to R43
Connections:
- net GND: now also Q18.1 (S), R44.2
- new net: D6.2 (A), M1.2 (-), Q18.3 (D)
- new net 24V: D6.1 (K), M1.1 (+)
- new net FAN: Q18.2 (G), R44.1
Other:
- moved on the sheet: R42, R43, R45, U13

Commit message: feat
Parts:
- removed M1: Fan, symbol Motor:Fan
- removed R44: 10k, symbol Device:R
- added D5: 1N5819, Diode_THT:D_DO-41_SOD81_P10.16mm_Horizontal, symbol Diode:1N5819
- added Q17: IRFZ44N, Package_TO_SOT_THT:TO-220-3_Vertical, symbol Transistor_FET:IRF540N
- added R41, R48: R, Resistor_THT:R_Axial_DIN0207_L6.3mm_D2.5mm_P7.62mm_Horizontal, symbol Device:R
- added R42, R43: 1k, Resistor_THT:R_Axial_DIN0207_L6.3mm_D2.5mm_P7.62mm_Horizontal, symbol Device:R
- added R46: 10k, Resistor_THT:R_Axial_DIN0207_L6.3mm_D2.5mm_P7.62mm_Horizontal, symbol Device:R
- added U13: PC817, Package_DIP:DIP-4_W7.62mm, symbol Isolator:PC817
- D6: footprint Diode_THT:D_DO-41_SOD81_P2.54mm_Vertical_KathodeUp -> Diode_THT:D_DO-41_SOD81_P10.16mm_Horizontal
- R44: renamed from R42; footprint (none) -> Resistor_THT:R_Axial_DIN0207_L6.3mm_D2.5mm_P7.62mm_Horizontal
- R45: renamed from R43; footprint (none) -> Resistor_THT:R_Axial_DIN0207_L6.3mm_D2.5mm_P7.62mm_Horizontal
- R47: renamed from R45; footprint (none) -> Resistor_THT:R_Axial_DIN0207_L6.3mm_D2.5mm_P7.62mm_Horizontal
- renumbered U13 to U14
Connections:
- net 24V: now also D5.1 (K), R42.1; no longer D6.1 (K)
- net 5V: now also D6.1 (K)
- net FAN: now also R41.1; no longer Q18.2 (G)
- net GND: now also Q17.3 (S), R43.2, R46.2, U13.2
- net BUZZER_EN_2: now reaches D6.2 (A), Q18.3 (D)
- net BUZZER_EN_2: now also R48.1
- new net: R41.2, U13.1
- new net: Q17.1 (G), R43.1, U13.3
- new net: R42.2, U13.4
- new net ALARM: Q18.2 (G), R46.1
- new net FAN-: D5.2 (A), Q17.2 (D)
- new net LED-: R48.2

Commit message: !feat
Parts:
- D5, D6: footprint Diode_THT:D_DO-41_SOD81_P10.16mm_Horizontal -> Diode_THT:D_DO-41_SOD81_P7.62mm_Horizontal
Changed lines of the file:
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@@
 			)
 		)
-		(property "Footprint" "Diode_THT:D_DO-41_SOD81_P10.16mm_Horizontal"
+		(property "Footprint" "Diode_THT:D_DO-41_SOD81_P7.62mm_Horizontal"
 			(at 161.925 114.3 0)
 			(effects
@@
 			)
 		)
-		(property "Footprint" "Diode_THT:D_DO-41_SOD81_P10.16mm_Horizontal"
+		(property "Footprint" "Diode_THT:D_DO-41_SOD81_P7.62mm_Horizontal"
 			(at 113.665 114.3 0)
 			(effects

Commit message: !feat
Connections:
- net BUZZER_EN_2: now also R48.2; no longer R48.1
- net GND: now also R45.2; no longer R45.1
- net LED-: now also R48.1; no longer R48.2
- net TX: now also R44.2, R45.1; no longer R44.1, R45.2
- net at U14.1 (RO): now also R44.1; no longer R44.2
Other:
- moved on the sheet: R44, R45, R48
Changed lines of the file:
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@@
 	(symbol
 		(lib_id "Device:R")
-		(at 162.56 119.38 90)
+		(at 162.56 119.38 270)
+		(mirror x)
 		(unit 1)
 		(exclude_from_sim no)
@@
 	(symbol
 		(lib_id "Device:R")
-		(at 118.11 69.85 180)
+		(at 118.11 69.85 0)
+		(mirror y)
 		(unit 1)
 		(exclude_from_sim no)
@@
 		(dnp no)
 		(property "Reference" "R44"
-			(at 120.65 68.5799 0)
+			(at 120.65 71.1201 0)
 			(effects
 				(font
@@
 		)
 		(property "Value" "10k"
-			(at 120.65 71.1199 0)
+			(at 120.65 68.5801 0)
 			(effects
 				(font
@@
 	(symbol
 		(lib_id "Device:R")
-		(at 118.11 80.01 180)
+		(at 118.11 80.01 0)
+		(mirror y)
 		(unit 1)
 		(exclude_from_sim no)
@@
 		(dnp no)
 		(property "Reference" "R45"
-			(at 120.65 78.7399 0)
+			(at 120.65 81.2801 0)
 			(effects
 				(font
@@
 		)
 		(property "Value" "18k"
-			(at 120.65 81.2799 0)
-			(effects
-				(font
+			(at 120.65 78.7401 0)
+			(effects
+				(font

Commit message: fix
Parts:
- R44: value 10k -> 1k
- R45: value 18k -> 1.5k
Changed lines of the file:
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@@
 			)
 		)
-		(property "Value" "10k"
+		(property "Value" "1k"
 			(at 120.65 68.5801 0)
 			(effects
@@
 			)
 		)
-		(property "Value" "18k"
+		(property "Value" "1.5k"
 			(at 120.65 78.7401 0)
 			(effects
