File: hardware/schematics/DIN_panel/DIN_panel.kicad_pcb (KiCad board)
At the start: 2 copper layers, 29 x 32 mm, 8 parts, among them J1 6P6C, J2 Buzzer enable, SW1 Reset

Commit message: chore
Other:
- board text added: "JLCJLCJLCJLC"
Changed lines of the file:
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@@
 			(outputformat 1)
 			(mirror no)
-			(drillshape 1)
+			(drillshape 0)
 			(scaleselection 1)
-			(outputdirectory "")
+			(outputdirectory "C:/Users/lozio/Desktop/DIN_panel/")
 		)
 	)
@@
 		)
 	)
+	(gr_text "JLCJLCJLCJLC"
+		(at 151 81 0)
+		(layer "B.SilkS")
+		(effects
+			(font
+				(size 0.8 0.8)
+				(thickness 0.16)
+				(bold yes)
+			)
+			(justify bottom mirror)
+		)
+	)
